File: hardware/kicad/watch/connectivity.kicad_sch (KiCad schematic)
At the start: 12 parts, among them U17 CXD5610GF, U19 HP5354.A, U21 BGA524N6, U23 BGA524N6, Y3 ECS-TXO-20CSMV4-260-AN-TR

Commit message: fah
Parts:
- added R32: 10k, Footprints:ERJS02_U02__0402_, symbol Symbols:ERJU02F1002X
Connections:
- net +1V8: now also R32.2
- net SPI_CS renamed CXD5610GF_CS
- net CXD5610GF_CS: now also R32.1
