File: hardware/kicad/watch/health.kicad_sch (KiCad schematic)
At the start: 39 parts, among them IC14 AS6223A-AWLT, J2 BIOZ2_POINT, J3 ECG_REF_P, J4 ECG_INP_P, J5 BIOZ4_POINT, U1 AS7058

Commit message: fah
Parts:
- added R33: 10k, Footprints:ERJS02_U02__0402_, symbol Symbols:ERJU02F1002X
Connections:
- net +1V8: now also R33.2
- net SPI_CS renamed AS7058_CSXN
- net AS7058_CSXN: now also R33.1
