File: hardware/kicad/watch/storage.kicad_sch (KiCad schematic)
At the start: 3 parts, among them U13 112J-TDAR-R01, U3 KLMCG4JETD-B041

Commit message: fah
Connections:
- no-connect marks 12 -> 13
Changed lines of the file:
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@@
+	)
+	(no_connect
+		(at 165.1 115.57)
 	)
 	(no_connect
